Commit message: [Edit] Update omo files related to jongmin workspace

File: omo_r1_description/urdf/omo_r1.urdf.g2.xacro (robot description, xacro)
@@ -159,10 +159,10 @@
     </inertial>
   </link>
-  <joint name="camera_joint" type="fixed">
+  <joint name="camera2_joint" type="fixed">
     <origin xyz="0.11 -0.0115 0.473" rpy="0 0.0 0"/>
     <parent link="base_link"/>
-    <child link="camera_link"/>
+    <child link="camera2_link"/>
   </joint>
-  <link name="camera_link">
+  <link name="camera2_link">
     <visual>
       <origin xyz="0 0 0.0" rpy="1.5758 0.0 1.5758"/>
@@ -179,15 +179,15 @@
     </collision>
   </link>
-  <joint name="camera_rgb_joint" type="fixed">
+  <joint name="camera2_rgb_joint" type="fixed">
     <origin xyz="0.03 0.0 0.0" rpy="0 0 0"/>
-    <parent link="camera_link"/>
-    <child link="camera_rgb_frame"/>
+    <parent link="camera2_link"/>
+    <child link="camera2_rgb_frame"/>
   </joint>
-  <link name="camera_rgb_frame"/>
-  <joint name="camera_rgb_optical_joint" type="fixed">
+  <link name="camera2_rgb_frame"/>
+  <joint name="camera2_rgb_optical_joint" type="fixed">
     <origin xyz="0 0 0" rpy="-1.57 0 -1.57"/>
-    <parent link="camera_rgb_frame"/>
-    <child link="camera_rgb_optical_frame"/>
+    <parent link="camera2_rgb_frame"/>
+    <child link="camera2_rgb_optical_frame"/>
   </joint>
-  <link name="camera_rgb_optical_frame"/>
+  <link name="camera2_rgb_optical_frame"/>
 </robot>
